File: DonationSafeBoard/donationsafeboard.kicad_pcb (KiCad board)
At the start: 2 copper layers, 5 parts

Commit message: put stuff on a board, add holes.
Parts:
- added REF**: MountingHole_4.5mm_Pad_TopBottom, MountingHole:MountingHole_4.5mm_Pad_TopBottom, F.Cu at (124.5, 110.2)
- added REF**: MountingHole_4.5mm_Pad_TopBottom, MountingHole:MountingHole_4.5mm_Pad_TopBottom, F.Cu at (155.2, 79.5)
- moved OUT1 31.4 mm to (152.0, 107.0)
- moved CASE_BUTTON1 23.7 mm to (139.0, 107.0)
- moved JUMPER1 23.3 mm to (139.0, 98.0)
- moved SWITCH1 22.3 mm to (143.0, 82.0)
- moved IN1 5.34 mm to (128.0, 82.0)
Routing:
- net Net-(CASE_BUTTON1-A): track 79.1 -> 35.4 mm
- net Net-(CASE_BUTTON1-B): track 68.9 -> 36.1 mm
- added copper zone on F.Cu, net GND
Other:
- board outline added: 40.5 x 40.5 mm

Commit message: logos, repo, version.
Parts:
- added REF**: KiCad-Logo2_6mm_SilkScreen, Symbol:KiCad-Logo2_6mm_SilkScreen, F.Cu at (132.0, 99.0)
Other:
- board text added: "$$$"
- board text added: "github.com/Naitotchi/DonationSafe-PowerBoard v1.0"
